Commit message: simplfied models

File: KitchenCounter/32354/mobility.urdf (robot description, URDF)
Before this commit: robot partnet_49ad167497a2af8c9672e39f89e4622e, 5 links, 4 joints
Links:
- removed link link_0
- removed link link_1
- removed link link_2
Joints:
- removed joint joint_0
- removed joint joint_1
- removed joint joint_2

File: KitchenCounter/32746/mobility.urdf (robot description, URDF)
Before this commit: robot partnet_ebc897217df591d73542091189dc62b5, 4 links, 3 joints
Links:
- removed link link_0
- removed link link_1
Joints:
- removed joint joint_0
- removed joint joint_1
