Commit message: all minifridges working

File: MiniFridge/10797/mobility.urdf (robot description, URDF)
Before this commit: robot partnet_6601ef650f03e000c49931aa7ca8fecb, 3 links, 2 joints
Links:
- added link handle; collision mesh filename=textured_objs/new-1-fixed.obj; visual mesh filename=textured_objs/new-1.obj
- link link_1: geometry collision mesh filename=textured_objs/new-2.obj; collision mesh filename=textured_objs/original-2.obj
Joints:
- added joint joint_handle: type fixed, parent link_1, child handle, origin xyz=0 0 0 rpy=0 0 0

File: MiniFridge/10849/mobility.urdf (robot description, URDF)
Before this commit: robot partnet_5b81d7830eabb7547c6e1fb05e1b9037, 3 links, 2 joints
Links:
- added link handle; collision mesh filename=textured_objs/new-1.obj; visual mesh filename=textured_objs/new-1.obj
- link link_0: geometry collision mesh filename=textured_objs/new-3.obj; collision mesh filename=textured_objs/new-4.obj
Joints:
- added joint joint_handle: type fixed, parent link_0, child handle, origin xyz=0 0 0, axis 0 1 0

File: MiniFridge/11178/mobility.urdf (robot description, URDF)
Before this commit: robot partnet_8ed3447275de7695149c1768202b4e64, 4 links, 3 joints
Links:
- added link handle_1; collision mesh filename=textured_objs/new-4-fixed.obj; visual mesh filename=textured_objs/new-4.obj
- added link handle_2; collision mesh filename=textured_objs/new-5.obj; visual mesh filename=textured_objs/new-5.obj
- link link_0: geometry collision mesh filename=textured_objs/new-8.obj; visual mesh filename=textured_objs/new-8.obj
- link link_1: geometry collision mesh filename=textured_objs/new-6.obj; visual mesh filename=textured_objs/new-6.obj
Joints:
- added joint joint_handle_1: type fixed, parent link_0, child handle_1, origin xyz=0 0 0, axis 0 -1 0
- added joint joint_handle_2: type fixed, parent link_1, child handle_2, origin xyz=0 0 0, axis 0 1 0

File: MiniFridge/11231/mobility.urdf (robot description, URDF)
Before this commit: robot partnet_a44c2110f646309bc7fb1a0a584939a5, 4 links, 3 joints
Links:
- added link handle_1; collision mesh filename=textured_objs/new-1-fixed.obj; visual mesh filename=textured_objs/new-1.obj
- added link handle_2; collision mesh filename=textured_objs/new-2.obj; visual mesh filename=textured_objs/new-2.obj
- link link_1: geometry collision mesh filename=textured_objs/new-3.obj; collision mesh filename=textured_objs/original-2.obj
- link link_2: geometry collision mesh filename=textured_objs/new-4.obj; visual mesh filename=textured_objs/new-4.obj
Joints:
- added joint joint_handle_1: type fixed, parent link_1, child handle_1, origin xyz=0 0 0, axis 0 1 0
- added joint joint_handle_2: type fixed, parent link_2, child handle_2, origin xyz=0 0 0, axis 0 -1 0

File: MiniFridge/11709/mobility.urdf (robot description, URDF)
Before this commit: robot partnet_f71397f01cab21ffaff7331733d1f0f5, 5 links, 4 joints
Links:
- added link link_0_handle; collision mesh filename=textured_objs/original-9-fixed.obj; visual mesh filename=textured_objs/original-9-fixed.obj
- added link link_1_handle; collision mesh filename=textured_objs/original-8-fixed.obj; visual mesh filename=textured_objs/original-8-fixed.obj
- added link link_2_handle; collision mesh filename=textured_objs/original-7-fixed.obj; visual mesh filename=textured_objs/original-7-fixed.obj
Joints:
- added joint joint_0_handle: type fixed, parent link_0, child link_0_handle, origin xyz=0 0 0, axis 0 -1 0
- added joint joint_1_handle: type fixed, parent link_1, child link_1_handle, origin xyz=0 0 0, axis 0 -1 0
- added joint joint_2_handle: type fixed, parent link_2, child link_2_handle, origin xyz=0 0 0, axis 0 -1 0

File: MiniFridge/12249/mobility.urdf (robot description, URDF)
Before this commit: robot partnet_3158fd17e409d38a732208e596b26ebc, 4 links, 3 joints
Links:
- link handle: geometry collision mesh filename=textured_objs/original-2-new.obj; visual mesh filename=textured_objs/original-2.obj

File: MiniFridge/12252/mobility.urdf (robot description, URDF)
Before this commit: robot partnet_7028b24b7d64efaf3194539af1047dcf, 3 links, 2 joints
Links:
- added link handle; collision mesh filename=textured_objs/original-16.obj; visual mesh filename=textured_objs/original-16.obj
- link link_0: geometry collision mesh filename=textured_objs/original-11.obj; collision mesh filename=textured_objs/original-12.obj
Joints:
- added joint joint_handle: type fixed, parent link_0, child handle, origin xyz=0 0 0, axis 0 1 0

Commit message: break first fridge

File: MiniFridge/10797/mobility.urdf (robot description, URDF)
Before this commit: robot partnet_6601ef650f03e000c49931aa7ca8fecb, 4 links, 3 joints
Links:
- link link_0: geometry collision mesh filename=textured_objs/new-0.obj; collision mesh filename=textured_objs/new-3-back.obj

Commit message: bulk

File: MiniFridge/10797/mobility.urdf (robot description, URDF)
Before this commit: robot partnet_6601ef650f03e000c49931aa7ca8fecb, 4 links, 3 joints
Links:
- link link_0: geometry collision mesh filename=textured_objs/new-0.obj; collision mesh filename=textured_objs/new-3-back-bulk.obj
