Commit message: breakdown

File: MiniFridge/11709/mobility.urdf (robot description, URDF)
Before this commit: robot partnet_f71397f01cab21ffaff7331733d1f0f5, 8 links, 7 joints
Links:
- link link_3: geometry collision mesh filename=textured_objs/original-1.obj; collision mesh filename=textured_objs/original-128-back.obj

File: MiniFridge/12249/mobility.urdf (robot description, URDF)
Before this commit: robot partnet_3158fd17e409d38a732208e596b26ebc, 4 links, 3 joints
Links:
- link link_1: geometry collision mesh filename=textured_objs/original-4-back.obj; collision mesh filename=textured_objs/original-4-bottom.obj

File: MiniFridge/12252/mobility.urdf (robot description, URDF)
Before this commit: robot partnet_7028b24b7d64efaf3194539af1047dcf, 4 links, 3 joints
Links:
- link link_1: geometry collision mesh filename=textured_objs/new-0.obj; collision mesh filename=textured_objs/new-1-back.obj
