Commit message: fix tomato and pepper urdf

File: Food/VeggieGreenPepper/mobility.urdf (robot description, URDF)
Before this commit: robot free3dmodels_veggie_green_pepper, 2 links, 1 joints
Joints:
- joint joint_1: origin xyz=0 0 0 rpy=0 0 -1.570796326794897 -> xyz=0 0 0 rpy=1.570796326794897 0 -1.570796326794897

File: Food/VeggieTomato/mobility.urdf (robot description, URDF)
Before this commit: robot free3dmodels_veggie_tomato, 2 links, 1 joints
Joints:
- joint joint_1: origin xyz=0 0 0 rpy=0 0 -1.570796326794897 -> xyz=0 0 0 rpy=1.570796326794897 0 -1.570796326794897
