Commit message: breakdown

File: MiniFridge/10849/mobility.urdf (robot description, URDF)
Before this commit: robot partnet_5b81d7830eabb7547c6e1fb05e1b9037, 4 links, 3 joints
Links:
- link link_1: geometry collision mesh filename=textured_objs/new-0.obj; collision mesh filename=textured_objs/new-2-back.obj

Commit message: bottom

File: MiniFridge/10849/mobility.urdf (robot description, URDF)
Before this commit: robot partnet_5b81d7830eabb7547c6e1fb05e1b9037, 4 links, 3 joints
Links:
- link link_1: geometry collision box size=1 .12 0.95; collision mesh filename=textured_objs/new-0.obj
