Commit message: seg fault

File: MiniFridge/11231/mobility.urdf (robot description, URDF)
Before this commit: robot partnet_a44c2110f646309bc7fb1a0a584939a5, 6 links, 5 joints
Links:
- link handle_1: geometry collision mesh filename=textured_objs/new-1-fixing.obj; visual mesh filename=textured_objs/new-1-fixing.obj

Commit message: gap in 11231

File: MiniFridge/11231/mobility.urdf (robot description, URDF)
Before this commit: robot partnet_a44c2110f646309bc7fb1a0a584939a5, 6 links, 5 joints
Links:
- link link_0: geometry collision mesh filename=textured_objs/new-0-bottom.obj; collision mesh filename=textured_objs/new-5-back.obj

Commit message: fridge instances

File: MiniFridge/11231/mobility.urdf (robot description, URDF)
Before this commit: robot partnet_a44c2110f646309bc7fb1a0a584939a5, 6 links, 5 joints
Links:
- link link_0: geometry collision box size=1.1 .1 0.7; collision mesh filename=textured_objs/new-0-bottom.obj
