Commit message: grasps on trays

File: Faucet/14/mobility.urdf (robot description, URDF)
Before this commit: robot partnet_2781a072e2645ccdedf1aa83ea962bc0, 9 links, 8 joints
Links:
- link link_0: geometry collision mesh filename=textured_objs/new-10.obj; collision mesh filename=textured_objs/original-7.obj
- link link_1: geometry collision mesh filename=textured_objs/new-6.obj; collision mesh filename=textured_objs/original-5.obj
- link link_2: geometry collision mesh filename=textured_objs/new-0.obj; collision mesh filename=textured_objs/original-3.obj
- link link_3: geometry collision mesh filename=textured_objs/new-12.obj; collision mesh filename=textured_objs/new-8.obj
- link link_nob_0: geometry collision mesh filename=textured_objs/new-11.obj; visual mesh filename=textured_objs/new-11.obj
- link link_nob_1: geometry collision mesh filename=textured_objs/new-7.obj; visual mesh filename=textured_objs/new-7.obj
- link link_nob_2: geometry visual mesh filename=textured_objs/new-14.obj
- link tube_head: geometry collision mesh filename=textured_objs/new-1.obj; visual mesh filename=textured_objs/new-1.obj
