Commit message: tray domain working

File: KitchenCounter/26608/mobility.urdf (robot description, URDF)
Before this commit: robot partnet_79b7bd0c910e833ba5dde908aa701435, 10 links, 9 joints
Joints:
- joint joint_7: limit lower=-0.12400000000000011 upper=0.1120000000000001 -> lower=0 upper=0.23199999999999998
