Commit message: long-horizon rearrangement working

File: Stapler/103100/mobility.urdf (robot description, URDF)
Before this commit: robot partnet_3800d2ab6bc278bcd5a3e6010c55b78e, 4 links, 3 joints
Joints:
- joint joint_0: origin xyz=0.0 0.021258419566391972 0.48796620307490224 -> xyz=0 0 0
- joint joint_1: origin xyz=0.0 -0.020562913603634957 -0.8268847886795407 -> xyz=0 0 0

File: Stapler/103104/mobility.urdf (robot description, URDF)
Before this commit: robot partnet_453034dc-b04a-4415-8c43-16d6d23c47b2, 4 links, 3 joints
Joints:
- joint joint_1: origin xyz=0.0 0.0677290172544402 -0.728057998017902 -> xyz=0 0 0

File: Stapler/103299/mobility.urdf (robot description, URDF)
Before this commit: robot partnet_f39912a4f0516fb897371d1e7cc637f3, 4 links, 3 joints
Joints:
- joint joint_1: origin xyz=0.0 -0.1533962566795296 -0.7771303494914226 -> xyz=0 0 0

File: Stapler/103307/mobility.urdf (robot description, URDF)
Before this commit: robot partnet_ue12a29d7-6d30-4159-ac11-3c6a058ad354, 4 links, 3 joints
Joints:
- joint joint_1: origin xyz=0.0 -0.06817607435527 -0.8689201614068358 -> xyz=0 0 0
