Commit message: full kitchen

File: Microwave/7265/mobility.urdf (robot description, URDF)
Before this commit: robot partnet_891f65c773939191c834958aed613724, 22 links, 21 joints
Joints:
- joint joint_0: limit lower=-0.5235987755982988 upper=1.3962634015954636 -> lower=0 upper=1.919862176; origin xyz=-0.6187850466966622 0 0.35921808895468765 -> xyz=-0.6187850466966622 0 0.35921808895468765 rpy=0 0.5235987755982988 0

File: OvenCounter/101808/mobility.urdf (robot description, URDF)
Before this commit: robot partnet_47c68395a5775e10d9deb3f829cc2475, 12 links, 11 joints
Joints:
- joint joint_9: origin xyz=0 0 0 rpy=1.570796326794897 0 -1.570796326794897 -> xyz=0 0 0 rpy=1.570796326794897 0 -1.500796326794897
