Commit message: sink pick

File: Sink/00003/mobility.urdf (robot description, URDF)
Before this commit: robot sink_003, 2 links, 1 joints
Links:
- added link sink_bottom; collision box size=0.38 .001 0.22; visual box size=0.38 .001 0.22
- link link_1: geometry collision mesh filename=sink_-x.obj; collision mesh filename=sink_-y.obj
Joints:
- added joint bottom_transform: type fixed, parent link_1, child sink_bottom, origin xyz=0 -0.05 0 rpy=0 0 0

File: Sink/00005/mobility.urdf (robot description, URDF)
Before this commit: robot sink_005, 2 links, 1 joints
Links:
- added link sink_bottom; collision box size=63 .001 56; visual box size=63 .001 56
- added link sink_bottom_2; collision box size=30 .001 48; visual box size=30 .001 48
- link link_1: geometry collision mesh filename=kitchen_sink_obj_back_left.obj; collision mesh filename=kitchen_sink_obj_back_right.obj
Joints:
- added joint bottom_transform: type fixed, parent link_1, child sink_bottom, origin xyz=16.5 -23.7 0 rpy=0 0 0
- added joint bottom_transform_2: type fixed, parent link_1, child sink_bottom_2, origin xyz=-33 -23.7 -4 rpy=0 0 0

File: Sink/100191/mobility.urdf (robot description, URDF)
Before this commit: robot partnet_549813be-3bd8-47dd-9a49-b51432b2f14c, 3 links, 2 joints
Links:
- removed link tray_bottom
- added link sink_bottom; collision mesh filename=textured_objs/original-1.obj; visual mesh filename=textured_objs/original-1.obj
Joints:
- joint joint_0: child tray_bottom -> sink_bottom

File: Sink/100501/mobility.urdf (robot description, URDF)
Before this commit: robot partnet_553c586e128708ae7649cce35db393a1, 3 links, 2 joints
Links:
- removed link tray_bottom
- added link sink_bottom; collision mesh filename=textured_objs/original-41.obj; visual mesh filename=textured_objs/original-41.obj
Joints:
- joint joint_0: child tray_bottom -> sink_bottom

File: Sink/100685/mobility.urdf (robot description, URDF)
Before this commit: robot partnet_u82f2a1a8-3a4b-4dd0-8fac-6679970a9b29, 3 links, 2 joints
Links:
- removed link tray_bottom
- added link sink_bottom; collision mesh filename=textured_objs/original-19-bottom.obj; visual mesh filename=textured_objs/original-19-bottom.obj
Joints:
- joint joint_0: child tray_bottom -> sink_bottom

File: Sink/101176/mobility.urdf (robot description, URDF)
Before this commit: robot partnet_e60bf49d6449cf37c5924a1a5d3043b0, 3 links, 2 joints
Links:
- removed link tray_bottom
- added link sink_bottom; collision mesh filename=textured_objs/original-22-bottom.obj; visual mesh filename=textured_objs/original-22-bottom-visual.obj
Joints:
- joint joint_0: child tray_bottom -> sink_bottom

File: Sink/102379/mobility.urdf (robot description, URDF)
Before this commit: robot partnet_3ac64751-e075-488d-9938-9123dc88b2b6-0, 9 links, 8 joints
Links:
- removed link basin_bottom
- added link sink_bottom; collision box size=1.26 .001 .84; visual box size=1.26 .001 .84
Joints:
- joint bottom_transform: child basin_bottom -> sink_bottom
