Commit message: sink collision

File: Sink/100685/mobility.urdf (robot description, URDF)
Before this commit: robot partnet_u82f2a1a8-3a4b-4dd0-8fac-6679970a9b29, 3 links, 2 joints
Links:
- link link_1: geometry collision mesh filename=textured_objs/original-19-back-collision.obj; collision mesh filename=textured_objs/original-19-bottom.obj
