Commit message: braiser breakdown

File: BraiserBody/100015/mobility.urdf (robot description, URDF)
Before this commit: robot partnet_11e7166d-8424-4edf-98cf-783b60539214-body, 3 links, 2 joints
Links:
- link link_1: geometry collision mesh filename=vhacd/original-19_vhacd_3083479662.obj; collision mesh filename=vhacd/original-22_vhacd_3081579112_part-0.obj

File: BraiserBody/100017/mobility.urdf (robot description, URDF)
Before this commit: robot partnet_1497ccf1ac032d35ce1decf313ece97f-body, 3 links, 2 joints
Links:
- link link_1: geometry collision mesh filename=../../assets/models/BraiserBody/100017/textured_objs/origin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; collision mesh filename=../../assets/models/BraiserBody/100017/textured_objs/origin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

File: BraiserBody/100021/mobility.urdf (robot description, URDF)
Before this commit: robot partnet_1fde7ce0a20f1502f54e1b6f41fdd78a-body, 3 links, 2 joints
Links:
- link link_1: geometry collision mesh filename=textured_objs/original-12.obj; collision mesh filename=textured_objs/original-13.obj

File: BraiserBody/100023/mobility.urdf (robot description, URDF)
Before this commit: robot partnet_2266db44d8411d909d0d74633db4834d-body, 3 links, 2 joints
Links:
- link link_1: geometry collision mesh filename=../../assets/models/BraiserBody/100023/textured_objs/origin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; collision mesh filename=../../assets/models/BraiserBody/100023/textured_objs/origin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

File: BraiserBody/100038/mobility.urdf (robot description, URDF)
Before this commit: robot partnet_7c4df032-d578-4bfb-958e-a7c7c31d655f-body, 3 links, 2 joints
Links:
- link link_1: geometry collision mesh filename=vhacd/original-10_vhacd_3090819690_part-0.obj; collision mesh filename=vhacd/original-10_vhacd_3090819690_part-1.obj

File: BraiserBody/100045/mobility.urdf (robot description, URDF)
Before this commit: robot partnet_d1cf7685d598f3929405d3391cbdb79b-body, 3 links, 2 joints
Links:
- link link_1: geometry collision mesh filename=textured_objs/original-8.obj; collision mesh filename=vhacd/original-10_vhacd_3086821992_part-0.obj
