Commit message: grasp lid

File: OvenCounter/101917/mobility.urdf (robot description, URDF)
Before this commit: robot partnet_8c2491e5245804d1ffc6e457221b9271, 10 links, 9 joints
Links:
- link link_8: geometry collision mesh filename=textured_objs/original-10.obj; collision mesh filename=textured_objs/original-113.obj
