Commit message: view in gym

File: OvenCounter/102001/mobility.urdf (robot description, URDF)
Before this commit: robot partnet_e69db4d377603b7d37b2bb75885cfc44, 11 links, 10 joints
Links:
- link link_9: geometry collision mesh filename=textured_objs/original-100.obj; collision mesh filename=textured_objs/original-101.obj
