Commit message: oven problem

File: OvenCounter/102018/mobility.urdf (robot description, URDF)
Before this commit: robot partnet_ef97ff5c1d6a00f2a760e402290727de, 8 links, 7 joints
Links:
- link link_6: geometry collision mesh filename=textured_objs/original-1.obj; collision mesh filename=textured_objs/original-100.obj
