Commit message: oven problem

File: OvenCounter/101921/mobility.urdf (robot description, URDF)
Before this commit: robot partnet_902f4ee7655514ba109dc73fee74b150, 11 links, 10 joints
Links:
- link link_9: geometry collision mesh filename=textured_objs/original-33.obj; collision mesh filename=textured_objs/original-34.obj
