Commit message: remove lid working

File: BraiserLid/100693/mobility.urdf (robot description, URDF)
Before this commit: robot partnet_d9560bfc0c051109f54e1b6f41fdd78a, 2 links, 1 joints
Links:
- link link_0: geometry collision mesh filename=textured_objs/original-7-new.obj; collision mesh filename=textured_objs/original-8-collision-2.obj

Commit message: lid problem

File: BraiserLid/100693/mobility.urdf (robot description, URDF)
Before this commit: robot partnet_d9560bfc0c051109f54e1b6f41fdd78a, 2 links, 1 joints
Links:
- added link handle_link; collision mesh filename=textured_objs/original-8-new.obj; visual mesh filename=textured_objs/original-8-fix.obj
- link link_0: geometry collision mesh filename=textured_objs/original-6-new.obj; collision mesh filename=textured_objs/original-7-new.obj
Joints:
- added joint handle_joint: type prismatic, parent link_0, child handle_link, origin xyz=0 0 0, axis 0 1 0, limit lower=0 upper=0.05
