Commit message: microwave problem

File: Microwave/_/7265/mobility.urdf (robot description, URDF)
Before this commit: robot partnet_891f65c773939191c834958aed613724, 22 links, 21 joints
Links:
- link link_0: geometry collision mesh filename=textured_objs/new-6.obj; collision mesh filename=textured_objs/original-3.obj
