Commit message: breakdown

File: MiniFridge/11178/mobility.urdf (robot description, URDF)
Before this commit: robot partnet_8ed3447275de7695149c1768202b4e64, 6 links, 5 joints
Links:
- link link_2: geometry collision mesh filename=textured_objs/new-0.obj; collision mesh filename=textured_objs/new-1.obj

File: MiniFridge/11231/mobility.urdf (robot description, URDF)
Before this commit: robot partnet_a44c2110f646309bc7fb1a0a584939a5, 6 links, 5 joints
Links:
- link link_0: geometry collision mesh filename=textured_objs/new-0.obj; collision mesh filename=textured_objs/new-5-back.obj

Commit message: fruit

File: MiniFridge/11178/mobility.urdf (robot description, URDF)
Before this commit: robot partnet_8ed3447275de7695149c1768202b4e64, 6 links, 5 joints
Links:
- link link_2: geometry collision mesh filename=textured_objs/new-0.obj; collision mesh filename=textured_objs/new-1.obj

File: MiniFridge/11231/mobility.urdf (robot description, URDF)
Before this commit: robot partnet_a44c2110f646309bc7fb1a0a584939a5, 6 links, 5 joints
Links:
- link link_0: geometry collision box size=1.1 .1 0.7; collision mesh filename=textured_objs/new-0-bottom.obj
