Commit message: sink bottom

File: Sink/101176/mobility.urdf (robot description, URDF)
Before this commit: robot partnet_e60bf49d6449cf37c5924a1a5d3043b0, 3 links, 2 joints
Links:
- link sink_bottom: geometry collision mesh filename=textured_objs/original-22-bottom.obj; visual box size=0.73 .001 1.1

File: Sink/102379/mobility.urdf (robot description, URDF)
Before this commit: robot partnet_3ac64751-e075-488d-9938-9123dc88b2b6-0, 9 links, 8 joints
Links:
- removed link basin
- removed link basin_base
- added link sink; collision mesh filename=textured_objs/original-47.obj; collision mesh filename=textured_objs/original-48.obj
- added link sink_base; collision mesh filename=base_objs/original-10.obj; collision mesh filename=base_objs/original-11.obj
Joints:
- joint bottom_transform: parent basin -> sink
- joint faucet_transform: parent basin -> sink
- joint joint_1: child basin_base -> sink_base
- joint joint_2: child basin -> sink; parent basin_base -> sink_base
- joint joint_collision_1: parent basin -> sink
- joint joint_collision_2: parent basin -> sink
- joint joint_collision_3: parent basin -> sink
- joint joint_collision_4: parent basin -> sink
