Commit message: dining table

File: DiningTable/25913/mobility.urdf (robot description, URDF)
Before this commit: robot partnet_90a1748069ca92df9667b9ba9d06c778, 5 links, 4 joints
Joints:
- joint joint_0: limit lower=0.0040000000000000036 upper=0.512 -> lower=0 upper=0.516; origin xyz=0 0 0 -> xyz=0.004 0 0
- joint joint_1: limit lower=-0.02400000000000002 upper=0.504 -> lower=0 upper=0.528; origin xyz=0 0 0 -> xyz=0 0 -0.024
- joint joint_2: limit lower=-0.07600000000000007 upper=0.42399999999999993 -> lower=0 upper=0.5; origin xyz=0 0 0 -> xyz=0 0 -0.076

File: DiningTable/28164/mobility.urdf (robot description, URDF)
Before this commit: robot partnet_bc4ba0bd86545f3fcc749dbc8c455b3f, 4 links, 3 joints
Joints:
- joint joint_1: limit lower=-0.28800000000000003 upper=0.08800000000000008 -> lower=0 upper=0.376; origin xyz=0 0 0 -> xyz=0 0 -0.288
