Commit message: kitchen skills

File: counter/urdf/kitchen_part_right_gen_convex.urdf (robot description, URDF)
Before this commit: robot kitchen_part_right, 53 links, 52 joints
Links:
- link chewie_door_left_handle: geometry collision mesh filename=../meshes/obj/handle_new.obj scale=1.0 1.0 1.0; visual mesh filename=../meshes/obj/handle_new.obj scale=1.0 1.0 1.0
- link chewie_door_left_link: geometry collision mesh filename=../meshes/obj/front_vertical_left.obj scale=1.0 1.0 1.0; visual mesh filename=../meshes/obj/front_vertical_left.obj scale=1.0 1.0 1.0
- link chewie_door_right_handle: geometry collision mesh filename=../meshes/obj/handle_new.obj scale=1.0 1.0 1.0; visual mesh filename=../meshes/obj/handle_new.obj scale=1.0 1.0 1.0
- link chewie_door_right_link: geometry collision mesh filename=../meshes/obj/front_vertical_right.obj scale=1.0 1.0 1.0; visual mesh filename=../meshes/obj/front_vertical_right.obj scale=1.0 1.0 1.0
- link dagger: geometry collision mesh filename=../meshes/obj/sektion_top_two_glass_new.obj scale=1.0 1.0 1.0; visual mesh filename=../meshes/obj/sektion_top_two_glass_new.obj scale=1.0 1.0 1.0
- link dagger_door_left_handle: geometry collision mesh filename=../meshes/obj/handle_new.obj scale=1.0 1.0 1.0; visual mesh filename=../meshes/obj/handle_new.obj scale=1.0 1.0 1.0
- link dagger_door_left_link: geometry collision mesh filename=../meshes/obj/front_vertical_left.obj scale=1.0 1.0 1.0; visual mesh filename=../meshes/obj/front_vertical_left.obj scale=1.0 1.0 1.0
- link dagger_door_right_handle: geometry collision mesh filename=../meshes/obj/handle_new.obj scale=1.0 1.0 1.0; visual mesh filename=../meshes/obj/handle_new.obj scale=1.0 1.0 1.0
- link dagger_door_right_link: geometry collision mesh filename=../meshes/obj/front_vertical_right.obj scale=1.0 1.0 1.0; visual mesh filename=../meshes/obj/front_vertical_right.obj scale=1.0 1.0 1.0
- link hitman_drawer_bottom: geometry collision box size=0.005 0.699 0.086; collision box size=0.512 0.004 0.086
- link hitman_drawer_handle_bottom: geometry collision mesh filename=../meshes/obj/handle.obj scale=1.0 1.0 1.0; visual mesh filename=../meshes/obj/handle.obj scale=1.0 1.0 1.0
- link hitman_drawer_handle_top: geometry collision mesh filename=../meshes/obj/handle.obj scale=1.0 1.0 1.0; visual mesh filename=../meshes/obj/handle.obj scale=1.0 1.0 1.0
- link hitman_drawer_top: geometry collision box size=0.005 0.699 0.086; collision box size=0.512 0.004 0.086
- link hitman_tmp: geometry collision box size=0.04 0.762 0.763; collision box size=0.61 0.019 0.763
- link indigo_door_left_link: geometry collision mesh filename=../meshes/obj/front_bottom_vertical_door.obj scale=1.0 1.0 1.0; visual mesh filename=../meshes/obj/front_bottom_vertical_door.obj scale=1.0 1.0 1.0
- link indigo_door_left_nob_link: geometry collision mesh filename=../meshes/obj/handle.obj scale=1.0 1.0 1.0; visual mesh filename=../meshes/obj/handle.obj scale=1.0 1.0 1.0
- link indigo_door_right_link: geometry collision mesh filename=../meshes/obj/front_bottom_vertical_door.obj scale=1.0 1.0 1.0; visual mesh filename=../meshes/obj/front_bottom_vertical_door.obj scale=1.0 1.0 1.0
- link indigo_door_right_nob_link: geometry collision mesh filename=../meshes/obj/handle.obj scale=1.0 1.0 1.0; visual mesh filename=../meshes/obj/handle.obj scale=1.0 1.0 1.0
- link indigo_drawer_bottom: geometry collision box size=0.004 0.699 0.086; collision box size=0.511 0.004 0.086
- link indigo_drawer_handle_bottom: geometry collision mesh filename=../meshes/obj/handle.obj scale=1.0 1.0 1.0; visual mesh filename=../meshes/obj/handle.obj scale=1.0 1.0 1.0
- link indigo_drawer_handle_top: geometry collision mesh filename=../meshes/obj/handle.obj scale=1.0 1.0 1.0; visual mesh filename=../meshes/obj/handle.obj scale=1.0 1.0 1.0
- link indigo_drawer_top: geometry collision box size=0.004 0.699 0.086; collision box size=0.511 0.004 0.086
- link indigo_tmp: geometry collision box size=0.04 0.762 0.763; collision box size=0.61 0.019 0.763
- link sektion: geometry collision mesh filename=../meshes/obj/sektion_top_three_new3_two.obj scale=1.0 1.0 1.0; visual mesh filename=../meshes/obj/sektion_top_three_new3_two.obj scale=1.0 1.0 1.0
- link walls: geometry collision mesh filename=../meshes/obj/walls.obj scale=1.0 1.0 1.0; visual mesh filename=../meshes/obj/walls.obj scale=1.0 1.0 1.0

Commit message: counter range

File: counter/urdf/kitchen_part_right_gen_convex.urdf (robot description, URDF)
Before this commit: robot kitchen_part_right, 53 links, 52 joints
Joints:
- joint chewie_door_left_joint: limit lower=-1.57 upper=0 effort=1000.0 velocity=0.1 -> lower=-2.34 upper=0 effort=1000.0 velocity=0.1
- joint chewie_door_right_joint: limit lower=0 upper=1.57 effort=1000.0 velocity=0.1 -> lower=0 upper=2.34 effort=1000.0 velocity=0.1

Commit message: handempty problem

File: counter/urdf/kitchen_part_right_gen_convex.urdf (robot description, URDF)
Before this commit: robot kitchen_part_right, 53 links, 52 joints
Joints:
- joint extractor_hood_transform: origin xyz=-0.14 0.415 0.37 rpy=0 0 0 -> xyz=-0.24 0.415 0.47 rpy=0 0 0

Commit message: counter visual

File: counter/urdf/kitchen_part_right_gen_convex.urdf (robot description, URDF)
Before this commit: robot kitchen_part_right, 53 links, 52 joints
Joints:
- joint extractor_hood_transform: origin xyz=-0.24 0.415 0.47 rpy=0 0 0 -> xyz=-0.21 0.415 0.47 rpy=0 0 0

Commit message: hitman_counter

File: counter/urdf/kitchen_part_right_gen_convex.urdf (robot description, URDF)
Before this commit: robot kitchen_part_right, 53 links, 52 joints
Links:
- link hitman_countertop: geometry collision box size=0.655 1.58 0.04; visual box size=0.655 1.58 0.04
Joints:
- joint hitman_countertop_transform: origin xyz=-0.04 -0.75 -0.02 rpy=0 0 0 -> xyz=-0.04 -0.8 -0.02 rpy=0 0 0
