Commit message: turkey visual

File: MeatTurkeyLeg/0001/mobility.urdf (robot description, URDF)
Before this commit: robot free3dmodels_meatturkeyleg, 2 links, 1 joints
Links:
- link link_1: geometry collision mesh filename=turkeyleg.obj; visual mesh filename=turkeyleg.obj

Commit message: reduce obj size

File: MeatTurkeyLeg/0001/mobility.urdf (robot description, URDF)
Before this commit: robot free3dmodels_meatturkeyleg, 2 links, 1 joints
Links:
- link link_1: geometry collision mesh filename=turkeyleg-reduced.obj; visual mesh filename=turkeyleg-reduced.obj
