Commit message: oven

File: Oven/01909/mobility.urdf (robot description, URDF)
Before this commit: robot partnet_8295e45a734c059d1f3d773b4af1f0c9, 8 links, 7 joints
Links:
- added link knob_link_1; collision mesh filename=textured_objs/original-12.obj; visual mesh filename=textured_objs/original-12.obj
- link link_1: geometry collision mesh filename=textured_objs/original-53.obj; visual mesh filename=textured_objs/original-53.obj
Joints:
- added joint knob_button_1: type fixed, parent link_5, child link_1, origin xyz=0.31708094673931356 0.7720745754611937 -0.15151306153341626, axis 0 0.19256852863983123 0.9812835277214688
- joint knob_joint_1: child link_1 -> knob_link_1; origin xyz=0.41708094673931356 0.7720745754611937 -0.15151306153341626 -> (none); parent link_5 -> link_1

Commit message: stove

File: Oven/01909/mobility.urdf (robot description, URDF)
Before this commit: robot partnet_8295e45a734c059d1f3d773b4af1f0c9, 9 links, 8 joints
Links:
- added link knob_link_3; collision mesh filename=textured_objs/original-8.obj; visual mesh filename=textured_objs/original-8.obj
- added link knob_link_4; collision mesh filename=textured_objs/original-6.obj; visual mesh filename=textured_objs/original-6.obj
- link link_3: geometry collision mesh filename=textured_objs/original-7.obj; visual mesh filename=textured_objs/original-7.obj
- link link_4: geometry collision mesh filename=textured_objs/original-49.obj; visual mesh filename=textured_objs/original-49.obj
Joints:
- added joint knob_button_3: type fixed, parent link_5, child link_3, origin xyz=-0.15347888005765334 0.7720745754611937 -0.15151306153341626, axis 0 0.19256852863983123 0.9812835277214688
- added joint knob_button_4: type fixed, parent link_5, child link_4, origin xyz=-0.2520335 0.7720745754611937 -0.15151306153341626, axis 0 0.19256852863983123 0.9812835277214688
- joint knob_joint_3: child link_3 -> knob_link_3; limit lower=-0.0 upper=5.672320068981571 -> lower=-0.0 upper=1.046666667; origin xyz=-0.15347888005765334 0.7720745754611937 -0.15151306153341626 -> (none); parent link_5 -> link_3
- joint knob_joint_4: child link_4 -> knob_link_4; limit lower=-6.283185307179586 upper=-0.6108652381980153 -> lower=-0.0 upper=1.046666667; origin xyz=-0.3520335 0.7720735939143407 -0.15153806521756305 -> (none); parent link_5 -> link_4

Commit message: rummy kitchen

File: Oven/01909/mobility.urdf (robot description, URDF)
Before this commit: robot partnet_8295e45a734c059d1f3d773b4af1f0c9, 11 links, 10 joints
Joints:
- joint knob_button_1: origin xyz=0.31708094673931356 0.7720745754611937 -0.15151306153341626 -> xyz=0.36708094673931356 0.8020745754611937 -0.16151306153341626
- joint knob_button_4: origin xyz=-0.2520335 0.7720745754611937 -0.15151306153341626 -> xyz=-0.3020335 0.8020745754611937 -0.16151306153341626

File: counter/urdf/kitchen_part_right_gen_convex.urdf (robot description, URDF)
Before this commit: robot kitchen_part_right, 53 links, 52 joints
Links:
- removed link indigo_door_left_nob_link
- removed link indigo_door_right_nob_link
- added link indigo_door_left_handle, mass 1.0; collision mesh filename=../meshes/obj/handle.obj scale=1.0 1.0 1.0; visual mesh filename=../meshes/obj/handle.obj scale=1.0 1.0 1.0
- added link indigo_door_right_handle, mass 1.0; collision mesh filename=../meshes/obj/handle.obj scale=1.0 1.0 1.0; visual mesh filename=../meshes/obj/handle.obj scale=1.0 1.0 1.0
Joints:
- joint indigo_door_left_nob_transform: child indigo_door_left_nob_link -> indigo_door_left_handle
- joint indigo_door_right_nob_transform: child indigo_door_right_nob_link -> indigo_door_right_handle
